Commit message: feat(slam): add rtabmap_ros

File: agv_pro_description/urdf/agv_pro.urdf (robot description, URDF)
Before this commit: robot AGV pro, 7 links, 6 joints
Links:
- added link ${namespace}camera_link
Joints:
- added joint ${namespace}camera_joint: type fixed, parent ${namespace}base_link, child ${namespace}camera_link, origin xyz=0.23191 0 0.14928 rpy=0 0 0

Commit message: fix(agv_pro_description): Fix missing imu_link

File: agv_pro_description/urdf/agv_pro.urdf (robot description, URDF)
Before this commit: robot AGV pro, 8 links, 7 joints
Links:
- added link ${namespace}imu_link
Joints:
- added joint ${namespace}imu_joint: type fixed, parent ${namespace}base_link, child ${namespace}imu_link, origin xyz=-0.17181 -0.0270532 0.14928 rpy=0 0 1.5707
